File: PCB_DESIGN/FINAL_PROJECT/Fpga.kicad_sch (KiCad schematic)
At the start: 12 parts, among them J1 Conn_01x06_Pin, U1 CA56-12CGKWA, U2 CA56-12CGKWA, U3 LFXP2-5E-5TN144

Commit message: Updated PCB
Parts:
- U1, U2: footprint Display_7Segment:CA56-12CGKWA -> Display_7Segment:KCSC02-107
Changed lines of the file:
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@@
 		)
 		(instances
-			(project "schemetics"
+			(project "FINAL_PROJECT"
 				(path "/047bd40c-18cc-4ecd-88f1-0eecd6e2e7c2/6caebfca-b986-4e80-be3c-3adf5503915c"
 					(reference "R6")
@@
 		)
 		(instances
-			(project "schemetics"
+			(project "FINAL_PROJECT"
 				(path "/047bd40c-18cc-4ecd-88f1-0eecd6e2e7c2/6caebfca-b986-4e80-be3c-3adf5503915c"
 					(reference "J1")
@@
 		)
 		(instances
-			(project "schemetics"
+			(project "FINAL_PROJECT"
 				(path "/047bd40c-18cc-4ecd-88f1-0eecd6e2e7c2/6caebfca-b986-4e80-be3c-3adf5503915c"
 					(reference "R4")
@@
 		)
 		(instances
-			(project "schemetics"
+			(project "FINAL_PROJECT"
 				(path "/047bd40c-18cc-4ecd-88f1-0eecd6e2e7c2/6caebfca-b986-4e80-be3c-3adf5503915c"
 					(reference "R1")
@@
 			)
 		)
-		(property "Footprint" "Display_7Segment:CA56-12CGKWA"
+		(property "Footprint" "Display_7Segment:KCSC02-107"
 			(at 165.1 74.93 0)
 			(effects
@@
 		)
 		(instances
-			(project "schemetics"
+			(project "FINAL_PROJECT"
 				(path "/047bd40c-18cc-4ecd-88f1-0eecd6e2e7c2/6caebfca-b986-4e80-be3c-3adf5503915c"
 					(reference "U2")
@@
 		)
 		(instances
-			(project "schemetics"
+			(project "FINAL_PROJECT"
 				(path "/047bd40c-18cc-4ecd-88f1-0eecd6e2e7c2/6caebfca-b986-4e80-be3c-3adf5503915c"
 					(reference "R3")
@@
 		)
 		(instances
-			(project "schemetics"
+			(project "FINAL_PROJECT"
 				(path "/047bd40c-18cc-4ecd-88f1-0eecd6e2e7c2/6caebfca-b986-4e80-be3c-3adf5503915c"
 					(reference "U3")
@@
 		)
 		(instances
-			(project "schemetics"
+			(project "FINAL_PROJECT"
 				(path "/047bd40c-18cc-4ecd-88f1-0eecd6e2e7c2/6caebfca-b986-4e80-be3c-3adf5503915c"
 					(reference "R5")
@@
 		)
 		(instances
-			(project "schemetics"
+			(project "FINAL_PROJECT"
 				(path "/047bd40c-18cc-4ecd-88f1-0eecd6e2e7c2/6caebfca-b986-4e80-be3c-3adf5503915c"
 					(reference "R7")
@@
 		)
 		(instances
-			(project "schemetics"
+			(project "FINAL_PROJECT"
 				(path "/047bd40c-18cc-4ecd-88f1-0eecd6e2e7c2/6caebfca-b986-4e80-be3c-3adf5503915c"
 					(reference "R2")
@@
 			)
 		)
-		(property "Footprint" "Display_7Segment:CA56-12CGKWA"
+		(property "Footprint" "Display_7Segment:KCSC02-107"
 			(at 76.2 80.01 0)
 			(effects
@@
 		)
 		(instances
-			(project "schemetics"
+			(project "FINAL_PROJECT"
 				(path "/047bd40c-18cc-4ecd-88f1-0eecd6e2e7c2/6caebfca-b986-4e80-be3c-3adf5503915c"
 					(reference "U1")
@@
 		)
 		(instances
-			(project "schemetics"
+			(project "FINAL_PROJECT"
 				(path "/047bd40c-18cc-4ecd-88f1-0eecd6e2e7c2/6caebfca-b986-4e80-be3c-3adf5503915c"
 					(reference "R8")
